File: pcb/esr_meter_rev_b/esr_meter_rev_b.kicad_pcb (KiCad board)
At the start: 2 copper layers, 68.7 x 78.2 mm, 88 parts, among them CON1 External power, P1 Cx+, P2 Cx, P3 Cx-, P4 9V battery, P5 uA connector, Q1 BC547, Q2 BC557, Q3 BC547, SW1 On/Off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

Commit message: Cosmetic changes to PCB.
Parts:
- REF**: value Screw_Type2 -> Screw_Type4
- REF** (x5): value Screw_Type2 -> Screw_Type4; footprint ESR_Meter_Footprints:Symbol_Screw_Type2_SilkscreenTop -> ESR_Meter_Footprints:Symbol_Screw_Type4_SilkscreenTop
- REF** (x6): value Screw_Type3 -> Screw_Type2; footprint ESR_Meter_Footprints:Symbol_Screw_Type3_SilkscreenTop -> ESR_Meter_Footprints:Symbol_Screw_Type2_SilkscreenTop
- moved REF** 1.17 mm to (184.3, 111.8)
- moved REF** 0.99 mm to (122.4, 111.9)
- moved REF** 0.54 mm to (155.7, 51.1)
Routing:
- net Net-(R21-Pad1): track 20.3 -> 22.9 mm
- net Net-(P5-Pad1): track 39.1 -> 41.6 mm
Other:
- board text added: "PCB designed by Dmitry Melnichansky 4X1MD"
- board text removed: "PCB designe by Dmitry Melnichansky 4X1mD"

Commit message: Corrected silkprints.
Parts:
- turned R5 to 90 degrees
