File: pcb/esr_meter_rev_b/esr_meter_rev_b.sch (KiCad schematic (older format))
At the start: 71 parts, among them CON1 External power, P1 Cx+, P2 Cx, P3 Cx-, P4 9V battery, P5 uA connector, Q1 BC547, Q2 BC557, Q3 BC547, SW1 On/Off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

Commit message: Minor update.
Other:
- moved on the sheet: R10, R9
